Commit message: dump

File: pybullet_sim/assets/wsg50/wsg50.urdf (robot description, URDF)
Before this commit: robot wsg_50, 5 links, 4 joints
Links:
- link finger_left: geometry collision box size=0.013 0.02 0.08; visual box size=0.013 0.02 0.08
- link finger_right: geometry collision box size=0.013 0.02 0.08; visual box size=0.013 0.02 0.08

Commit message: change wsg50 urdf to have finger joint frame at center of finger link

File: pybullet_sim/assets/wsg50/wsg50.urdf (robot description, URDF)
Before this commit: robot wsg_50, 5 links, 4 joints
Joints:
- joint guide_joint_finger_left: origin xyz=0 0 0.023 rpy=0 0 0 -> xyz=-0.0051 0 0.113 rpy=0 0 0
- joint guide_joint_finger_right: origin xyz=0 0 0.023 rpy=0 0 0 -> xyz=0.0051 0 0.113 rpy=0 0 0
